File: loco3.kicad_sch (KiCad schematic)
At the start: 15 parts, among them J1 6P6C, J2 6P6C, J3 6P6C, U1 NE555D

Commit message: feat: Switch to disable LEDs
Parts:
- added SW1: SW_DIP_x02, Button_Switch_THT:SW_DIP_SPSTx02_Slide_9.78x7.26mm_W7.62mm_P2.54mm, symbol Switch:SW_DIP_x02
- C1: footprint (none) -> Capacitor_SMD:C_0603_1608Metric; LCSC (none) -> C57112
- C2: footprint (none) -> Capacitor_SMD:C_0603_1608Metric; LCSC (none) -> C14663
- C3: footprint (none) -> Capacitor_SMD:C_0805_2012Metric; LCSC (none) -> C15850
- D1, D2: value D -> BAT54J; footprint (none) -> Diode_SMD:D_SOD-323_HandSoldering; LCSC (none) -> C191023
- D3: LCSC (none) -> C2286
- D4: LCSC (none) -> C2297
- R1: footprint (none) -> Resistor_SMD:R_0603_1608Metric; LCSC (none) -> C25804
- R2, R4: footprint (none) -> Resistor_SMD:R_0603_1608Metric; LCSC (none) -> C22975
- R3: footprint (none) -> Resistor_SMD:R_0603_1608Metric; LCSC (none) -> C4190
- U1: LCSC (none) -> C7593
Connections:
- net VCC: now also SW1.1, SW1.2; no longer C2.1, R2.1, R3.1, U1.4 (R), U1.8 (VCC)
- new net: R3.1, SW1.4, U1.4 (R), U1.8 (VCC)
- new net: C2.1, R2.1, SW1.3
Other:
- moved on the sheet: C1, C2, C3, D2, D3, D4, R1, R2, R3, R4, U1

Commit message: WIP
Parts:
- J1, J3: footprint Samacsys:955012611 -> Snapeda:A-2004-1-4-LP-N-R_ASSMANN_A-2004-1-4-LP-N-R
- J2: footprint Snapeda:CUI_CRJ025-1-TH -> Snapeda:A-2014-1-4-N-T-R_ASSMANN_A-2014-1-4-N-T-R
Changed lines of the file:
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@@
 			)
 		)
-		(property "Footprint" "Samacsys:955012611"
+		(property "Footprint" "Snapeda:A-2004-1-4-LP-N-R_ASSMANN_A-2004-1-4-LP-N-R"
 			(at 172.085 60.96 90)
 			(effects
@@
 			)
 		)
-		(property "Footprint" "Snapeda:CUI_CRJ025-1-TH"
+		(property "Footprint" "Snapeda:A-2014-1-4-N-T-R_ASSMANN_A-2014-1-4-N-T-R"
 			(at 141.605 60.96 90)
 			(effects
@@
 			)
 		)
-		(property "Footprint" "Samacsys:955012611"
+		(property "Footprint" "Snapeda:A-2004-1-4-LP-N-R_ASSMANN_A-2004-1-4-LP-N-R"
 			(at 109.855 60.96 90)
 			(effects

Commit message: feat: Change LED resistors to decrease brightness
Parts:
- R2: value 2k -> 22k; LCSC C22975 -> C31850
- R4: value 2k -> 27k; LCSC C22975 -> C22967
Changed lines of the file:
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@@
 			)
 		)
-		(property "Value" "2k"
+		(property "Value" "22k"
 			(at 101.6 120.6499 0)
 			(effects
@@
 			)
 		)
-		(property "LCSC" "C22975"
+		(property "LCSC" "C31850"
 			(at 99.06 119.38 0)
 			(effects
@@
 			)
 		)
-		(property "Value" "2k"
+		(property "Value" "27k"
 			(at 186.69 123.1899 0)
 			(effects
@@
 			)
 		)
-		(property "LCSC" "C22975"
+		(property "LCSC" "C22967"
 			(at 184.15 121.92 0)
 			(effects
